Commit message: Fixed package errors for reorganisation

File: src/myrobot_description/urdf/myrobot.urdf.xacro (robot description, xacro)
@@ -3,5 +3,5 @@
     xmlns:xacro="http://www.ros.org/wiki/xacro">
     <!-- SUB-COMPONENTS -->
-    <xacro:include filename="$(find myrobot_gazebo)/urdf/myrobot_wheel.urdf.xacro" />
+    <xacro:include filename="$(find myrobot_description)/urdf/myrobot_wheel.urdf.xacro" />
     <!-- PROPERTIES -->
     <xacro:property name="M_PI" value="3.14159"/>
@@ -18,5 +18,5 @@
     <xacro:property name="use_drive_controller" value="true" />
     <!-- PLUGINS -->
-    <xacro:include filename="$(find myrobot_gazebo)/urdf/myrobot.gazebo.xacro" />
+    <xacro:include filename="$(find myrobot_description)/urdf/myrobot.gazebo.xacro" />
     <!-- PARTS -->
     <link name="robot_footprint"></link>
@@ -110,5 +110,5 @@
             <origin xyz="0.0 0.0 0.0" rpy="0.0 0.0 0.0"/>
             <geometry>
-                <mesh filename="package://myrobot_gazebo/meshes/hokuyo.dae" />
+                <mesh filename="package://myrobot_description/meshes/hokuyo.dae" />
             </geometry>
             <material name="">
